Commit message: Rover visual model done!

File: rover_ws/src/rover_description/urdf/rover.urdf (robot description, URDF)
Before this commit: robot rover, 13 links, 12 joints
Links:
- removed link antenna_link
- removed link drivewhl_l_front_link
- removed link drivewhl_l_middle_link
- removed link drivewhl_l_rear_link
- removed link drivewhl_r_front_link
- removed link drivewhl_r_middle_link
- removed link drivewhl_r_rear_link
- added link pole_link; visual box size=0.04 0.08 1.2
- added link wheel_left_front_link; visual cylinder length=0.2 radius=0.15
- added link wheel_left_middle_link; visual cylinder length=0.2 radius=0.15
- added link wheel_left_rear_link; visual cylinder length=0.2 radius=0.15
- added link wheel_right_front_link; visual cylinder length=0.2 radius=0.15
- added link wheel_right_middle_link; visual cylinder length=0.2 radius=0.15
- added link wheel_right_rear_link; visual cylinder length=0.2 radius=0.15
- link base_link: geometry visual box size=0.4 0.5 0.15
Joints:
- removed joint antenna_joint
- removed joint drivewhl_l_front_joint
- removed joint drivewhl_l_middle_joint
- removed joint drivewhl_l_rear_joint
- removed joint drivewhl_r_front_joint
- removed joint drivewhl_r_middle_joint
- removed joint drivewhl_r_rear_joint
- added joint pole_joint: type fixed, parent base_link, child pole_link, origin xyz=0.22 0 0.525 rpy=0 0 0
- added joint wheel_left_front_joint: type fixed, parent base_link, child wheel_left_front_link, origin xyz=0.835 0.44999999999999996 -0.15 rpy=0 0 0
- added joint wheel_left_middle_joint: type fixed, parent base_link, child wheel_left_middle_link, origin xyz=0.135 0.44999999999999996 -0.15 rpy=0 0 0
- added joint wheel_left_rear_joint: type fixed, parent base_link, child wheel_left_rear_link, origin xyz=-0.565 0.44999999999999996 -0.15 rpy=0 0 0
- added joint wheel_right_front_joint: type fixed, parent base_link, child wheel_right_front_link, origin xyz=0.835 -0.44999999999999996 -0.15 rpy=0 0 0
- added joint wheel_right_middle_joint: type fixed, parent base_link, child wheel_right_middle_link, origin xyz=0.135 -0.44999999999999996 -0.15 rpy=0 0 0
- added joint wheel_right_rear_joint: type fixed, parent base_link, child wheel_right_rear_link, origin xyz=-0.565 -0.44999999999999996 -0.15 rpy=0 0 0

File: rover_ws/src/rover_description/urdf/rover.xacro (robot description, xacro)
@@ -4,13 +4,20 @@
   <!-- Based on the sensor joints from the turtlebot3 gps, modified to match our config -->
   <!-- Rover constants -->
-  <xacro:property name="base_width" value="1.0"/>
-  <xacro:property name="base_length" value="1.5"/>
-  <xacro:property name="base_height" value="0.5"/>
-  <xacro:property name="wheel_radius" value="0.2"/>
-  <xacro:property name="wheel_width" value="0.1"/>
-  <xacro:property name="wheel_xoff" value="0.6"/>
-  <xacro:property name="wheel_ygap" value="0.05"/>
-  <xacro:property name="wheel_zoff" value="0.2"/>
-  <xacro:property name="antenna_length" value="0.5"/>
+  <xacro:property name="base_width" value="0.5"/>
+  <xacro:property name="base_length" value="0.4"/>
+  <xacro:property name="base_height" value="0.15"/>
+  <!-- How far back the rover carriage is compared to the center of the middle wheel -->
+  <xacro:property name="base_offset_x" value="0.135"/>
+  <xacro:property name="wheel_radius" value="0.15"/>
+  <xacro:property name="wheel_width" value="0.2"/>
+  <!-- How far the center of the front wheel is from the center of the middle wheel -->
+  <xacro:property name="wheel_xoff" value="0.7"/>
+  <!-- How far the center of the wheel is from the outside of the base -->
+  <xacro:property name="wheel_ygap" value="0.1"/>
+  <!-- How far down the center of the wheels are from the base center -->
+  <xacro:property name="wheel_zoff" value="0.15"/>
+  <xacro:property name="pole_length" value="0.04"/>
+  <xacro:property name="pole_width" value="0.08"/>
+  <xacro:property name="pole_height" value="1.2"/>
   <!-- Rover base -->
   <link name="base_link">
@@ -40,19 +47,19 @@
       <parent link="base_link"/>
       <child link="${prefix}_link"/>
-      <origin xyz="${x_reflect*(wheel_xoff - (wheel_pos * (base_length/3)))} ${y_reflect*(base_width/2+wheel_ygap)} ${-wheel_zoff}" rpy="0 0 0"/>
+      <origin xyz="${x_reflect*(wheel_xoff*(wheel_pos-1))+base_offset_x} ${y_reflect*(base_width/2+wheel_ygap+wheel_width/2)} ${-wheel_zoff}" rpy="0 0 0"/>
     </joint>
   </xacro:macro>
   <!-- Rover wheels -->
-  <xacro:wheel prefix="drivewhl_l_front" x_reflect="-1" y_reflect="1" wheel_pos="0"/>
-  <xacro:wheel prefix="drivewhl_l_middle" x_reflect="-1" y_reflect="1" wheel_pos="1"/>
-  <xacro:wheel prefix="drivewhl_l_rear" x_reflect="-1" y_reflect="1" wheel_pos="2"/>
-  <xacro:wheel prefix="drivewhl_r_front" x_reflect="-1" y_reflect="-1" wheel_pos="0"/>
-  <xacro:wheel prefix="drivewhl_r_middle" x_reflect="-1" y_reflect="-1" wheel_pos="1"/>
-  <xacro:wheel prefix="drivewhl_r_rear" x_reflect="-1" y_reflect="-1" wheel_pos="2"/>
+  <xacro:wheel prefix="wheel_left_front" x_reflect="-1" y_reflect="1" wheel_pos="0"/>
+  <xacro:wheel prefix="wheel_left_middle" x_reflect="-1" y_reflect="1" wheel_pos="1"/>
+  <xacro:wheel prefix="wheel_left_rear" x_reflect="-1" y_reflect="1" wheel_pos="2"/>
+  <xacro:wheel prefix="wheel_right_front" x_reflect="-1" y_reflect="-1" wheel_pos="0"/>
+  <xacro:wheel prefix="wheel_right_middle" x_reflect="-1" y_reflect="-1" wheel_pos="1"/>
+  <xacro:wheel prefix="wheel_right_rear" x_reflect="-1" y_reflect="-1" wheel_pos="2"/>
   <!-- Antenna pole -->
-  <link name="antenna_link">
+  <link name="pole_link">
     <visual>
       <geometry>
-        <cylinder radius="0.01" length="${antenna_length}"/>
+        <box size="${pole_length} ${pole_width} ${pole_height}"/>
       </geometry>
       <material name="White">
@@ -61,8 +68,8 @@
     </visual>
   </link>
-  <joint name="antenna_joint" type="fixed">
+  <joint name="pole_joint" type="fixed">
     <parent link="base_link"/>
-    <child link="antenna_link"/>
-    <origin xyz="0 0 0.5" rpy="0 0 0"/>
+    <child link="pole_link"/>
+    <origin xyz="${base_length/2+pole_length/2} 0 ${pole_height/2-base_height/2}" rpy="0 0 0"/>
   </joint>
   <!-- Sensors -->

Commit message: Added full urdf for rover

File: rover_ws/src/rover_description/urdf/rover.urdf (robot description, URDF)
Before this commit: robot rover, 13 links, 12 joints
Joints:
- joint aruco_cam_joint: origin xyz=0 0 0 rpy=0 0 0 -> xyz=0.02 0 0.1 rpy=0 0 0; parent base_link -> pole_link
- joint gps_joint: origin xyz=0 0 0 rpy=0 0 0 -> xyz=-0.2 0 0.075 rpy=0 0 0
- joint unilidar_lidar_joint: origin xyz=-0.064 0 0.122 rpy=0 0 0 -> xyz=0.12000000000000001 0 -0.05 rpy=3.141592653589793 0 0; parent base_link -> pole_link
- joint zed2_camera_joint: origin xyz=-0.064 0 0.122 rpy=0 0 0 -> xyz=0.02 0 0.05 rpy=0 0 0; parent base_link -> pole_link

File: rover_ws/src/rover_description/urdf/rover.xacro (robot description, xacro)
@@ -77,21 +77,18 @@
     <parent link="base_link"/>
     <child link="gps_link"/>
-    <!-- TODO: Update the gps position - Nelson -->
-    <origin xyz="0 0 0" rpy="0 0 0"/>
+    <origin xyz="${-base_length/2} 0 ${base_height/2}" rpy="0 0 0"/>
   </joint>
   <link name="gps_link"/>
   <joint name="aruco_cam_joint" type="fixed">
-    <parent link="base_link"/>
+    <parent link="pole_link"/>
     <child link="aruco_cam_link"/>
-    <!-- TODO: Update the aruco cam position - Nelson -->
-    <origin xyz="0 0 0" rpy="0 0 0"/>
+    <origin xyz="${pole_length/2} 0 0.1" rpy="0 0 0"/>
   </joint>
   <link name="aruco_cam_link"/>
   <!-- https://github.com/unitreerobotics/unilidar_sdk/blob/main/unitree_lidar_ros2/src/unitree_lidar_ros2/README.md -->
   <joint name="unilidar_lidar_joint" type="fixed">
-    <parent link="base_link"/>
+    <parent link="pole_link"/>
     <child link="unilidar_lidar"/>
-    <!-- TODO: Update the lidar position - Nelson -->
-    <origin xyz="-0.064 0 0.122" rpy="0 0 0"/>
+    <origin xyz="${pole_length/2+0.1} 0 -0.05" rpy="${pi} 0 0"/>
   </joint>
   <link name="unilidar_lidar"/>
@@ -105,8 +102,7 @@
   <!-- https://www.stereolabs.com/docs/ros2/020_zed-node#transform-frames -->
   <joint name="zed2_camera_joint" type="fixed">
-    <parent link="base_link"/>
+    <parent link="pole_link"/>
     <child link="zed2_camera_link"/>
-    <!-- TODO: Update the camera position - Nelson -->
-    <origin xyz="-0.064 0 0.122" rpy="0 0 0"/>
+    <origin xyz="${pole_length/2} 0 0.05" rpy="0 0 0"/>
   </joint>
   <link name="zed2_camera_link"/>
