Commit message: zed frame naming update

File: rover_ws/src/rover_description/urdf/rover.urdf.xacro (robot description, xacro)
@@ -99,9 +99,9 @@
   <link name="unilidar_imu"/>
   <!-- https://www.stereolabs.com/docs/ros2/140_ros2-robot-integration -->
-  <joint name="zed2_camera_joint" type="fixed">
+  <joint name="zed_camera_joint" type="fixed">
     <parent link="pole_link"/>
     <child link="zed2_camera_link"/>
     <origin xyz="${pole_length/2} 0 0.05" rpy="0 0 0"/>
   </joint>
-  <link name="zed2_camera_link"/>
+  <link name="zed_camera_link"/>
 </robot>

Commit message: Quick fix

File: rover_ws/src/rover_description/urdf/rover.urdf.xacro (robot description, xacro)
@@ -101,5 +101,5 @@
   <joint name="zed_camera_joint" type="fixed">
     <parent link="pole_link"/>
-    <child link="zed2_camera_link"/>
+    <child link="zed_camera_link"/>
     <origin xyz="${pole_length/2} 0 0.05" rpy="0 0 0"/>
   </joint>

Commit message: Zed and lidar calibration. Frames look good in RVIZ with the point clouds lined up

File: rover_ws/src/rover_description/urdf/rover.urdf.xacro (robot description, xacro)
@@ -88,20 +88,20 @@
   <joint name="unilidar_lidar_joint" type="fixed">
     <parent link="pole_link"/>
-    <child link="unilidar_lidar"/>
-    <origin xyz="${pole_length/2+0.1} 0 -0.05" rpy="${pi} 0 0"/>
+    <child link="unilidar_mount"/>
+    <origin xyz="${pole_length/2+0.1} 0 -0.05" rpy="0 ${pi/2} 0"/>
   </joint>
-  <link name="unilidar_lidar"/>
-  <joint name="unilidar_imu_joint" type="fixed">
+  <link name="unilidar_mount"/>
+  <!-- <joint name="unilidar_imu_joint" type="fixed">
     <parent link="unilidar_lidar"/>
     <child link="unilidar_imu"/>
     <origin xyz="0 0 0" rpy="0 0 0"/>
   </joint>
-  <link name="unilidar_imu"/>
+  <link name="unilidar_imu"/> -->
   <!-- https://www.stereolabs.com/docs/ros2/140_ros2-robot-integration -->
   <joint name="zed_camera_joint" type="fixed">
     <parent link="pole_link"/>
-    <child link="zed_camera_link"/>
+    <child link="zed_camera_mount"/>
     <origin xyz="${pole_length/2} 0 0.05" rpy="0 0 0"/>
   </joint>
-  <link name="zed_camera_link"/>
+  <link name="zed_camera_mount"/>
 </robot>

Commit message: TODO fixes

File: rover_ws/src/rover_description/urdf/rover.urdf.xacro (robot description, xacro)
@@ -2,5 +2,4 @@
 <robot name="rover" xmlns:xacro="http://ros.org/wiki/xacro">
   <!-- Created by Nelson Durrant, Mar 2025 -->
-  <!-- TODO: Make this more accurate -->
   <!-- Rover constants -->
   <xacro:property name="base_width" value="0.5"/>
@@ -83,5 +82,5 @@
     <parent link="pole_link"/>
     <child link="aruco_cam_link"/>
-    <origin xyz="${pole_length/2} 0 0.1" rpy="0 0 0"/>
+    <origin xyz="${pole_length/2+0.1} 0 0.1" rpy="0 0 0"/>
   </joint>
   <link name="aruco_cam_link"/>
@@ -90,18 +89,14 @@
     <parent link="pole_link"/>
     <child link="unilidar_mount"/>
+    <!-- the 'zed_lidar_calibrate' node handles the mount to sensor transform -->
     <origin xyz="${pole_length/2+0.1} 0 -0.05" rpy="0 ${pi/2} 0"/>
   </joint>
   <link name="unilidar_mount"/>
-  <!-- <joint name="unilidar_imu_joint" type="fixed">
-    <parent link="unilidar_lidar"/>
-    <child link="unilidar_imu"/>
-    <origin xyz="0 0 0" rpy="0 0 0"/>
-  </joint>
-  <link name="unilidar_imu"/> -->
   <!-- https://www.stereolabs.com/docs/ros2/140_ros2-robot-integration -->
   <joint name="zed_camera_joint" type="fixed">
     <parent link="pole_link"/>
     <child link="zed_camera_mount"/>
-    <origin xyz="${pole_length/2} 0 0.05" rpy="0 0 0"/>
+    <!-- the 'zed_lidar_calibrate' node handles the mount to sensor transform -->
+    <origin xyz="${pole_length/2+0.1} 0 0.05" rpy="0 0 0"/>
   </joint>
   <link name="zed_camera_mount"/>

Commit message: The ZED now manages odom->base_link

File: rover_ws/src/rover_description/urdf/rover.urdf.xacro (robot description, xacro)
@@ -2,4 +2,5 @@
 <robot name="rover" xmlns:xacro="http://ros.org/wiki/xacro">
   <!-- Created by Nelson Durrant, Mar 2025 -->
+  <!-- This model uses zed_camera_link as the top-level frame instead of base_link -->
   <!-- https://docs.nav2.org/setup_guides/urdf/setup_urdf.html#writing-the-urdf -->
   <!-- Rover constants -->
@@ -69,7 +70,7 @@
   </link>
   <joint name="pole_joint" type="fixed">
-    <parent link="base_link"/>
-    <child link="pole_link"/>
-    <origin xyz="${base_length/2+pole_length/2} 0 ${pole_height/2-base_height/2}" rpy="0 0 0"/>
+    <parent link="pole_link"/>
+    <child link="base_link"/>
+    <origin xyz="${-base_length/2-pole_length/2} 0 ${-pole_height/2+base_height/2}" rpy="0 0 0"/>
   </joint>
   <!-- Sensors -->
@@ -80,25 +81,17 @@
   </joint>
   <link name="gps_link"/>
-  <joint name="aruco_cam_joint" type="fixed">
-    <parent link="pole_link"/>
-    <child link="aruco_cam_link"/>
-    <origin xyz="${pole_length/2+0.1} 0 0.1" rpy="0 0 0"/>
-  </joint>
-  <link name="aruco_cam_link"/>
   <!-- https://github.com/unitreerobotics/unilidar_sdk/blob/main/unitree_lidar_ros2/src/unitree_lidar_ros2/README.md -->
   <joint name="unilidar_lidar_joint" type="fixed">
     <parent link="pole_link"/>
-    <child link="unilidar_mount"/>
-    <!-- the 'zed_lidar_calibrate' node handles the mount to sensor transform -->
+    <child link="unilidar_link"/>
     <origin xyz="${pole_length/2+0.1} 0 -0.05" rpy="0 ${pi/2} 0"/>
   </joint>
-  <link name="unilidar_mount"/>
+  <link name="unilidar_link"/>
   <!-- https://www.stereolabs.com/docs/ros2/140_ros2-robot-integration -->
   <joint name="zed_camera_joint" type="fixed">
-    <parent link="pole_link"/>
-    <child link="zed_camera_mount"/>
-    <!-- the 'zed_lidar_calibrate' node handles the mount to sensor transform -->
-    <origin xyz="${pole_length/2+0.1} 0 0.05" rpy="0 0 0"/>
+    <parent link="zed_camera_link"/>
+    <child link="base_link"/>
+    <origin xyz="${-pole_length/2-0.1} 0 -0.05" rpy="0 0 0"/>
   </joint>
-  <link name="zed_camera_mount"/>
+  <link name="zed_camera_link"/>
 </robot>

Commit message: EKF working!

File: rover_ws/src/rover_description/urdf/rover.urdf.xacro (robot description, xacro)
@@ -91,5 +91,5 @@
   <joint name="zed_camera_joint" type="fixed">
     <parent link="zed_camera_link"/>
-    <child link="base_link"/>
+    <child link="pole_link"/>
     <origin xyz="${-pole_length/2-0.1} 0 -0.05" rpy="0 0 0"/>
   </joint>

Commit message: ZED now angled in URDF

File: rover_ws/src/rover_description/urdf/rover.urdf.xacro (robot description, xacro)
@@ -93,5 +93,5 @@
     <parent link="zed_camera_link"/>
     <child link="pole_link"/>
-    <origin xyz="${-pole_length/2-0.1} 0 -0.05" rpy="0 0 0"/>
+    <origin xyz="${-pole_length/2-0.1} 0 -0.05" rpy="0 -0.2 0"/>
   </joint>
   <link name="zed_camera_link"/>

Commit message: Added new rover model

File: rover_ws/src/rover_description/urdf/rover.urdf.xacro (robot description, xacro)
@@ -5,11 +5,4 @@
     since the ZED publishes the odom->zed_camera_link transform instead of odom->base_link.
     https://docs.nav2.org/setup_guides/urdf/setup_urdf.html#writing-the-urdf -->
-  <!-- NOTE: Future teams might decide to try and get this custom model running in the Gazebo
-    simulation instead of the modified turtlebot3. We think the turtlebot3 is pretty great stand-in
-    for our rover sensor-wise, but for resources on getting this model hooked better into our control
-    system (other than just providing static transforms) and simulating it in Gazebo, see:
-    https://docs.nav2.org/setup_guides/urdf/setup_urdf.html
-    https://docs.nav2.org/setup_guides/odom/setup_odom_gz_classic.html
-    https://docs.nav2.org/setup_guides/sensors/setup_sensors_gz_classic.html -->
   <!-- Rover constants -->
   <xacro:property name="base_width" value="0.5"/>
@@ -29,4 +22,6 @@
   <xacro:property name="pole_width" value="0.08"/>
   <xacro:property name="pole_height" value="1.2"/>
+  <!-- Gazebo simulation plugins -->
+  <xacro:include filename="$(find rover_description)/urdf/rover.gazebo.xacro" />
   <!-- Rover base -->
   <link name="base_link">
@@ -39,7 +34,37 @@
       </material>
     </visual>
+    <collision>
+        <geometry>
+            <box size="${base_length} ${base_width} ${base_height}"/>
+        </geometry>
+    </collision>
+    <inertial>
+        <mass value="10"/>
+        <inertia ixx="1.0" ixy="0.0" ixz="0.0" iyy="1.0" iyz="0.0" izz="1.0"/>
+    </inertial>
   </link>
+  <!-- Rocker assembly function -->
+  <xacro:macro name="rocker_assembly" params="prefix y_reflect">
+    <link name="${prefix}_rocker_link">
+      <inertial>
+        <mass value="2"/>
+        <origin xyz="0 0 0" rpy="0 0 0"/>
+        <inertia ixx="0.1" ixy="0" ixz="0" iyy="0.1" iyz="0" izz="0.1"/>
+      </inertial>
+    </link>
+    <joint name="${prefix}_rocker_joint" type="revolute">
+      <parent link="base_link"/>
+      <child link="${prefix}_rocker_link"/>
+      <origin xyz="${base_offset_x} ${y_reflect*(base_width/2+wheel_ygap+wheel_width/2)} ${-wheel_zoff}" rpy="0 0 0"/>
+      <axis xyz="0 1 0"/>
+      <limit lower="-${pi/6}" upper="${pi/6}" effort="100" velocity="1.0"/>
+      <dynamics damping="0.5"/>
+    </joint>
+  </xacro:macro>
+  <!-- Rocker assemblies -->
+  <xacro:rocker_assembly prefix="left" y_reflect="1"/>
+  <xacro:rocker_assembly prefix="right" y_reflect="-1"/>
   <!-- Rover wheels function -->
-  <xacro:macro name="wheel" params="prefix x_reflect y_reflect wheel_pos">
+  <xacro:macro name="wheel" params="prefix x_reflect y_reflect wheel_pos y_reflect_prefix">
     <link name="${prefix}_link">
       <visual>
@@ -52,18 +77,28 @@
         </material>
       </visual>
+      <collision>
+        <origin xyz="0 0 0" rpy="${pi/2} 0 0"/>
+        <geometry>
+            <cylinder radius="${wheel_radius}" length="${wheel_width}"/>
+        </geometry>
+      </collision>
+      <inertial>
+        <mass value="1"/>
+        <inertia ixx="0.009" ixy="0.0" ixz="0.0" iyy="0.011" iyz="0.0" izz="0.009"/>
+      </inertial>
     </link>
-    <joint name="${prefix}_joint" type="fixed">
-      <parent link="base_link"/>
+    <joint name="${prefix}_joint" type="continuous">
+      <parent link="${y_reflect_prefix}_rocker_link"/>
       <child link="${prefix}_link"/>
-      <origin xyz="${x_reflect*(wheel_xoff*(wheel_pos-1))+base_offset_x} ${y_reflect*(base_width/2+wheel_ygap+wheel_width/2)} ${-wheel_zoff}" rpy="0 0 0"/>
+      <origin xyz="${x_reflect*(wheel_xoff*(wheel_pos-1))} 0 0" rpy="0 0 0"/>      <axis xyz="0 1 0"/>
     </joint>
   </xacro:macro>
   <!-- Rover wheels -->
-  <xacro:wheel prefix="wheel_left_front" x_reflect="-1" y_reflect="1" wheel_pos="0"/>
-  <xacro:wheel prefix="wheel_left_middle" x_reflect="-1" y_reflect="1" wheel_pos="1"/>
-  <xacro:wheel prefix="wheel_left_rear" x_reflect="-1" y_reflect="1" wheel_pos="2"/>
-  <xacro:wheel prefix="wheel_right_front" x_reflect="-1" y_reflect="-1" wheel_pos="0"/>
-  <xacro:wheel prefix="wheel_right_middle" x_reflect="-1" y_reflect="-1" wheel_pos="1"/>
-  <xacro:wheel prefix="wheel_right_rear" x_reflect="-1" y_reflect="-1" wheel_pos="2"/>
+  <xacro:wheel prefix="wheel_left_middle"  x_reflect="-1" y_reflect="1" wheel_pos="1" y_reflect_prefix="left"/>
+  <xacro:wheel prefix="wheel_right_middle" x_reflect="-1" y_reflect="-1" wheel_pos="1" y_reflect_prefix="right"/>
+  <xacro:wheel prefix="wheel_left_front"   x_reflect="-1" y_reflect="1" wheel_pos="0" y_reflect_prefix="left"/>
+  <xacro:wheel prefix="wheel_left_rear"    x_reflect="-1" y_reflect="1" wheel_pos="2" y_reflect_prefix="left"/>
+  <xacro:wheel prefix="wheel_right_front"  x_reflect="-1" y_reflect="-1" wheel_pos="0" y_reflect_prefix="right"/>
+  <xacro:wheel prefix="wheel_right_rear"   x_reflect="-1" y_reflect="-1" wheel_pos="2" y_reflect_prefix="right"/>
   <!-- Antenna pole -->
   <link name="pole_link">
@@ -76,4 +111,13 @@
       </material>
     </visual>
+    <collision>
+        <geometry>
+            <box size="${pole_length} ${pole_width} ${pole_height}"/>
+        </geometry>
+    </collision>
+    <inertial>
+        <mass value="1"/>
+        <inertia ixx="1.0" ixy="0.0" ixz="0.0" iyy="1.0" iyz="0.0" izz="1.0"/>
+    </inertial>
   </link>
   <joint name="pole_joint" type="fixed">
@@ -88,12 +132,22 @@
     <origin xyz="${-base_length/2} 0 ${base_height/2}" rpy="0 0 0"/>
   </joint>
-  <link name="gps_link"/>
-  <!-- https://github.com/unitreerobotics/unilidar_sdk/blob/main/unitree_lidar_ros2/src/unitree_lidar_ros2/README.md -->
-  <joint name="unilidar_lidar_joint" type="fixed">
+  <link name="gps_link">
+    <inertial>
+        <mass value="0.1"/>
+        <inertia ixx="0.1" ixy="0.0" ixz="0.0" iyy="0.1" iyz="0.0" izz="0.1"/>
+    </inertial>
+  </link>
+  <!-- LiDAR (used by the simulator) -->
+  <joint name="lidar_lidar_joint" type="fixed">
     <parent link="pole_link"/>
-    <child link="unilidar_link"/>
-    <origin xyz="${pole_length/2+0.1} 0 -0.05" rpy="0 ${pi/2} 0"/>
+    <child link="lidar_link"/>
+    <origin xyz="${pole_length/2+0.1} 0 -0.05" rpy="0 0 0"/>
   </joint>
-  <link name="unilidar_link"/>
+  <link name="lidar_link">
+    <inertial>
+        <mass value="0.1"/>
+        <inertia ixx="0.1" ixy="0.0" ixz="0.0" iyy="0.1" iyz="0.0" izz="0.1"/>
+    </inertial>
+  </link>
   <!-- https://www.stereolabs.com/docs/ros2/140_ros2-robot-integration -->
   <joint name="zed_camera_joint" type="fixed">
@@ -102,4 +156,5 @@
     <origin xyz="${-pole_length/2-0.1} 0 -0.05" rpy="0 -0.2 0"/>
   </joint>
+  <!-- As the top of the URDF tree, this can't have an intertial attribute -->
   <link name="zed_camera_link"/>
 </robot>

Commit message: Small fixes for URDF

File: rover_ws/src/rover_description/urdf/rover.urdf.xacro (robot description, xacro)
@@ -155,5 +155,5 @@
     <parent link="zed_camera_link"/>
     <child link="pole_link"/>
-    <origin xyz="${-pole_length/2-0.1} 0 -0.05" rpy="0 -0.2 0"/>
+    <origin xyz="${-pole_length/2-0.1} 0 -0.05" rpy="0 -0.1 0"/>
   </joint>
   <!-- NOTE: As the top of the URDF tree, this can't have an intertial attribute -->
