Commit message: It can drive around now, still a couple bugs with aruco detection and spin search to squash

File: rover_ws/src/rover_description/urdf/rover.gazebo.xacro (robot description, xacro)
@@ -8,23 +8,20 @@
   <!--                      GAZEBO PLUGINS                                 -->
   <!-- =================================================================== -->
-  <!-- Differential Drive Plugin for controlling the rover -->
-  <gazebo>
-    <plugin name="gazebo_ros_diff_drive" filename="libgazebo_ros_diff_drive.so">
-      <update_rate>30</update_rate>
-      <!-- Wheel and joint parameters -->
+  <!-- Kind of a hacky way to get all-wheel drive in sim, but hey it works -->
+  <!-- Middle wheel drive plugin -->
+  <gazebo>
+    <plugin name="gazebo_ros_diff_drive_middle" filename="libgazebo_ros_diff_drive.so">
+      <update_rate>30</update_rate>
       <left_joint>wheel_left_middle_joint</left_joint>
       <right_joint>wheel_right_middle_joint</right_joint>
       <wheel_separation>${base_width + 2*wheel_ygap + wheel_width}</wheel_separation>
       <wheel_diameter>${2*wheel_radius}</wheel_diameter>
-      <!-- Physics limits -->
-      <max_wheel_torque>2000</max_wheel_torque>
-      <max_wheel_acceleration>100.0</max_wheel_acceleration>
-      <!-- Frame and TF parameters -->
+      <max_wheel_torque>200</max_wheel_torque>
+      <max_wheel_acceleration>10.0</max_wheel_acceleration>
       <odometry_frame>odom</odometry_frame>
       <robot_base_frame>zed_camera_link</robot_base_frame>
-      <publish_odom>true</publish_odom>
+      <publish_odom>true</publish_odom> <!-- only publish here! -->
       <publish_odom_tf>false</publish_odom_tf>
       <publish_wheel_tf>false</publish_wheel_tf>
-      <!-- ROS 2 specific topic remapping -->
       <ros>
         <remapping>cmd_vel:=cmd_vel_mux</remapping>
@@ -33,4 +30,44 @@
     </plugin>
   </gazebo>
+  <!-- Front wheel drive plugin -->
+  <gazebo>
+    <plugin name="gazebo_ros_diff_drive_front" filename="libgazebo_ros_diff_drive.so">
+      <update_rate>30</update_rate>
+      <left_joint>wheel_left_front_joint</left_joint>
+      <right_joint>wheel_right_front_joint</right_joint>
+      <wheel_separation>${base_width + 2*wheel_ygap + wheel_width}</wheel_separation>
+      <wheel_diameter>${2*wheel_radius}</wheel_diameter>
+      <max_wheel_torque>200</max_wheel_torque>
+      <max_wheel_acceleration>10.0</max_wheel_acceleration>
+      <odometry_frame>odom</odometry_frame>
+      <robot_base_frame>zed_camera_link</robot_base_frame>
+      <publish_odom>false</publish_odom>
+      <publish_odom_tf>false</publish_odom_tf>
+      <publish_wheel_tf>false</publish_wheel_tf>
+      <ros>
+        <remapping>cmd_vel:=cmd_vel_mux</remapping>
+      </ros>
+    </plugin>
+  </gazebo>
+  <!-- Rear wheel drive plugin -->
+  <gazebo>
+    <plugin name="gazebo_ros_diff_drive_rear" filename="libgazebo_ros_diff_drive.so">
+      <update_rate>30</update_rate>
+      <left_joint>wheel_left_rear_joint</left_joint>
+      <right_joint>wheel_right_rear_joint</right_joint>
+      <wheel_separation>${base_width + 2*wheel_ygap + wheel_width}</wheel_separation>
+      <wheel_diameter>${2*wheel_radius}</wheel_diameter>
+      <max_wheel_torque>200</max_wheel_torque>
+      <max_wheel_acceleration>10.0</max_wheel_acceleration>
+      <odometry_frame>odom</odometry_frame>
+      <robot_base_frame>zed_camera_link</robot_base_frame>
+      <publish_odom>false</publish_odom>
+      <publish_odom_tf>false</publish_odom_tf>
+      <publish_wheel_tf>false</publish_wheel_tf>
+      <ros>
+        <remapping>cmd_vel:=cmd_vel_mux</remapping>
+      </ros>
+    </plugin>
+  </gazebo>
   <!-- Joint State Publisher for all wheel joints -->
   <gazebo>
@@ -40,4 +77,6 @@
       </ros>
       <update_rate>30</update_rate>
+      <joint_name>left_rocker_joint</joint_name>
+      <joint_name>right_rocker_joint</joint_name>
       <joint_name>wheel_left_front_joint</joint_name>
       <joint_name>wheel_left_middle_joint</joint_name>
@@ -59,6 +98,4 @@
   </gazebo>
   <!-- Macro for wheel physics and appearance -->
-  <!-- IMPORTANT! The physics is way easier when you just drive with two wheels -->
-  <!-- The others have no friction at all -->
   <xacro:macro name="wheel_gazebo" params="prefix mu1:=1.0 mu2:=1.0">
     <gazebo reference="${prefix}_link">
@@ -68,8 +105,8 @@
     </gazebo>
   </xacro:macro>
-  <xacro:wheel_gazebo prefix="wheel_left_front"  mu1="0.1" mu2="0.1"/>
-  <xacro:wheel_gazebo prefix="wheel_left_rear"   mu1="0.1" mu2="0.1"/>
-  <xacro:wheel_gazebo prefix="wheel_right_front" mu1="0.1" mu2="0.1"/>
-  <xacro:wheel_gazebo prefix="wheel_right_rear"  mu1="0.1" mu2="0.1"/>
+  <xacro:wheel_gazebo prefix="wheel_left_front"  mu1="50.0" mu2="50.0"/>
+  <xacro:wheel_gazebo prefix="wheel_left_rear"   mu1="50.0" mu2="50.0"/>
+  <xacro:wheel_gazebo prefix="wheel_right_front" mu1="50.0" mu2="50.0"/>
+  <xacro:wheel_gazebo prefix="wheel_right_rear"  mu1="50.0" mu2="50.0"/>
   <xacro:wheel_gazebo prefix="wheel_left_middle"  mu1="200.0" mu2="200.0"/>
   <xacro:wheel_gazebo prefix="wheel_right_middle" mu1="200.0" mu2="200.0"/>

File: rover_ws/src/rover_description/urdf/rover.urdf.xacro (robot description, xacro)
@@ -58,5 +58,5 @@
       <origin xyz="${base_offset_x} ${y_reflect*(base_width/2+wheel_ygap+wheel_width/2)} ${-wheel_zoff}" rpy="0 0 0"/>
       <axis xyz="0 1 0"/>
-      <limit lower="-${pi/6}" upper="${pi/6}" effort="100" velocity="1.0"/>
+      <limit lower="-${pi/6}" upper="${pi/36}" effort="100" velocity="1.0"/>
       <dynamics damping="0.5"/>
     </joint>

Commit message: Fix for sim camera coordinate frame

File: rover_ws/src/rover_description/urdf/rover.gazebo.xacro (robot description, xacro)
@@ -184,5 +184,5 @@
       <plugin name="intel_realsense_r200_depth_driver" filename="libgazebo_ros_camera.so">
         <camera_name>intel_realsense_r200_depth</camera_name>
-        <frame_name>zed_camera_link</frame_name> <!-- TODO: Figure this out -->
+        <frame_name>intel_realsense_link</frame_name>
       </plugin>
     </sensor>

File: rover_ws/src/rover_description/urdf/rover.urdf.xacro (robot description, xacro)
@@ -150,5 +150,18 @@
     </inertial>
   </link>
+  <!-- Intel Realsense Camera (used by the simulator) -->
+  <joint name="intel_realsense_joint" type="fixed">
+    <parent link="zed_camera_link"/>
+    <child link="intel_realsense_link"/>
+    <origin xyz="0 0 0" rpy="${-pi/2} 0 ${-pi/2}"/>
+  </joint>
+  <link name="intel_realsense_link">
+    <inertial>
+        <mass value="0.1"/>
+        <inertia ixx="0.1" ixy="0.0" ixz="0.0" iyy="0.1" iyz="0.0" izz="0.1"/>
+    </inertial>
+  </link>
   <!-- ZED Camera -->
+  <!-- The ZED manages its own internal TF tree -->
   <!-- https://www.stereolabs.com/docs/ros2/140_ros2-robot-integration -->
   <joint name="zed_camera_joint" type="fixed">

Commit message: Simplified to just the depth camera

File: rover_ws/src/rover_description/urdf/rover.gazebo.xacro (robot description, xacro)
@@ -130,5 +130,5 @@
         </position_sensing>
       </gps>
-      <plugin name="my_gps_plugin" filename="libgazebo_ros_gps_sensor.so">
+      <plugin name="turtlebot3_gps" filename="libgazebo_ros_gps_sensor.so">
         <ros>
           <remapping>~/out:=/gps/fix</remapping>
@@ -137,41 +137,5 @@
     </sensor>
   </gazebo>
-  <!-- LiDAR Sensor (from turtlebot3, only in sim) -->
-  <gazebo reference="lidar_link">
-    <sensor name="hls_lfcd_lds" type="ray">
-      <always_on>true</always_on>
-      <visualize>false</visualize>
-      <pose>0 0 0 0 0 0</pose>
-      <update_rate>5</update_rate>
-      <ray>
-        <scan>
-          <horizontal>
-            <samples>360</samples>
-            <resolution>1.0</resolution>
-            <min_angle>0.0</min_angle>
-            <max_angle>6.28</max_angle>
-          </horizontal>
-        </scan>
-        <range>
-          <min>0.12</min>
-          <max>3.5</max>
-          <resolution>0.015</resolution>
-        </range>
-        <noise>
-          <type>gaussian</type>
-          <mean>0.0</mean>
-          <stddev>0.01</stddev>
-        </noise>
-      </ray>
-      <plugin name="turtlebot3_laserscan" filename="libgazebo_ros_ray_sensor.so">
-        <ros>
-            <remapping>~/out:=scan</remapping>
-        </ros>
-        <output_type>sensor_msgs/LaserScan</output_type>
-        <frame_name>lidar_link</frame_name>
-      </plugin>
-    </sensor>
-  </gazebo>
-  <!-- Depth Camera Sensor (from turtlebot3, only in sim)-->
+  <!-- Depth Camera (from turtlebot3, only in sim)-->
   <!-- In real life, we'll use the ZED 2 camera, not the Intel Realsense -->
   <gazebo reference="zed_camera_link">
@@ -185,4 +149,7 @@
         <camera_name>intel_realsense_r200_depth</camera_name>
         <frame_name>intel_realsense_link</frame_name>
+        <ros>
+          <remapping>~/points:=/zed/zed_node/point_cloud/cloud_registered</remapping>
+        </ros>
       </plugin>
     </sensor>
@@ -239,5 +206,5 @@
         <ros>
           <remapping>~/out:=/zed/zed_node/imu/data</remapping>
-          </ros>
+        </ros>
       </plugin>
     </sensor>

File: rover_ws/src/rover_description/urdf/rover.urdf.xacro (robot description, xacro)
@@ -126,5 +126,5 @@
     <origin xyz="${-base_length/2-pole_length/2} 0 ${-pole_height/2+base_height/2}" rpy="0 0 0"/>
   </joint>
-  <!-- Sensors -->
+  <!-- GPS Sensor -->
   <joint name="gps_joint" type="fixed">
     <parent link="base_link"/>
@@ -133,16 +133,4 @@
   </joint>
   <link name="gps_link">
-    <inertial>
-        <mass value="0.1"/>
-        <inertia ixx="0.1" ixy="0.0" ixz="0.0" iyy="0.1" iyz="0.0" izz="0.1"/>
-    </inertial>
-  </link>
-  <!-- LiDAR (used by the simulator) -->
-  <joint name="lidar_lidar_joint" type="fixed">
-    <parent link="pole_link"/>
-    <child link="lidar_link"/>
-    <origin xyz="${pole_length/2+0.1} 0 -0.05" rpy="0 0 0"/>
-  </joint>
-  <link name="lidar_link">
     <inertial>
         <mass value="0.1"/>
