Commit message: Added colors to CougUV URDF

File: rover_ws/src/cougars/coug_description/urdf/couguv.urdf.xacro (robot description, xacro)
@@ -22,4 +22,10 @@
   <material name="White">
     <color rgba="1 1 1 1"/>
+  </material>
+  <material name="Blue">
+    <color rgba="0.196 0.6 0.8 1"/>
+  </material>
+  <material name="Gray">
+    <color rgba="0.5 0.5 0.5 1"/>
   </material>
   <!-- Function to generate fins -->
@@ -48,5 +54,5 @@
         <cylinder radius="${base_radius}" length="${base_length-2*base_radius}"/>
       </geometry>
-      <material name="White"/>
+      <material name="Blue"/>
     </visual>
   </link>
@@ -93,5 +99,5 @@
         <sphere radius="${base_radius}"/>
       </geometry>
-      <material name="White"/>
+      <material name="Blue"/>
     </visual>
   </link>
@@ -108,5 +114,5 @@
         <cylinder radius="${base_radius*0.9}" length="${2*base_radius}"/>
       </geometry>
-      <material name="White"/>
+      <material name="Gray"/>
     </visual>
   </link>
